File: efm32core.sch (EAGLE design)
At the start: 7 parts

Commit message: do cleanups
Parts:
- removed SJ1: (no value), SparkFun_mod:SOLDERJUMPER_2WAYT
- removed U$34: FE10-2W_MIRROR, con-lsta:FE10-2W_MIRROR
Connections:
- removed net 5V: SJ1.3, U$34.18
- removed net VMCU_3V3: SJ1.1, U$34.2
- net CS: no longer U$34.10
- net DISP_ENABLE: no longer U$34.14
- net EXTCOMIN: no longer U$34.7
- net EXTMODE: no longer U$34.12
- net GND: no longer U$34.1
- net MOSI_SI: no longer U$34.4
- net SCLK: no longer U$34.8
- net VCC: no longer SJ1.2
Other:
- note added: "MCU"
- moved on the sheet: U$7A, U$7C, U$7E, U$7F, U$7PWR
Changed lines of the file:
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@@
 <?xml version="1.0" encoding="utf-8"?>
 <!DOCTYPE eagle SYSTEM "eagle.dtd">
-<eagle version="6.5.0">
+<eagle version="6.3">
 <drawing>
 <settings>
@@
 <setting verticaltext="up"/>
 </settings>
-<grid distance="0.1" unitdist="inch" unit="inch" style="lines" multiple="1" display="yes" altdistance="0.01" altunitdist="inch" altunit="inch"/>
+<grid distance="0.1" unitdist="inch" unit="inch" style="lines" multiple="1" display="no" altdistance="0.01" altunitdist="inch" altunit="inch"/>
 <layers>
 <layer number="1" name="Top" color="4" fill="1" visible="no" active="no"/>
@@
 <part name="FRAME1" library="frames" deviceset="A3L-LOC" device=""/>
 <part name="U$31" library="sharp_mem_lcd" deviceset="SHARP_MEM_LCD" device=""/>
-<part name="U$34" library="con-lsta" deviceset="FE10-2W_MIRROR" device=""/>
 <part name="C3" library="rcl" deviceset="C-EU" device="C0402K" value="1uF"/>
 <part name="C2" library="rcl" deviceset="C-EU" device="C0402K" value="100nF"/>
 <part name="C1" library="rcl" deviceset="C-EU" device="C0402K" value="100nF"/>
-<part name="P+2" library="supply1" deviceset="VCC" device=""/>
-<part name="SUPPLY1" library="supply2" deviceset="GND" device=""/>
 <part name="P+4" library="supply1" deviceset="VCC" device=""/>
 <part name="SUPPLY3" library="supply2" deviceset="GND" device=""/>
-<part name="SJ1" library="SparkFun_mod" deviceset="SOLDERJUMPER_2WAY" device="T"/>
 <part name="U$7" library="EnergyMicro" deviceset="EFM32LG332F256" device=""/>
 </parts>
@@
 <wire x1="190.5" y1="134.62" x2="190.5" y2="256.54" width="0.1524" layer="97" style="shortdash"/>
 <text x="15.24" y="241.3" size="3.81" layer="97">Expansion Header Connector</text>
-<text x="205.74" y="238.76" size="3.81" layer="97">Display</text>
+<text x="205.74" y="243.84" size="3.81" layer="97">Display</text>
 <text x="344.17" y="20.574" size="2.54" layer="94" font="vector">Librae</text>
 <wire x1="5.08" y1="134.62" x2="190.5" y2="134.62" width="0.1524" layer="97"/>
 <wire x1="190.5" y1="134.62" x2="381" y2="134.62" width="0.1524" layer="97"/>
+<text x="261.62" y="15.24" size="3.81" layer="97">MCU</text>
 </plain>
 <instances>
 <instance part="FRAME1" gate="G$1" x="0" y="0"/>
 <instance part="U$31" gate="G$1" x="302.26" y="177.8"/>
-<instance part="U$34" gate="G$1" x="83.82" y="175.26"/>
 <instance part="C3" gate="G$1" x="254" y="162.56" rot="R180"/>
 <instance part="C2" gate="G$1" x="243.84" y="162.56" rot="R180"/>
 <instance part="C1" gate="G$1" x="233.68" y="162.56" rot="R180"/>
-<instance part="P+2" gate="VCC" x="109.22" y="200.66"/>
-<instance part="SUPPLY1" gate="GND" x="68.58" y="160.02"/>
 <instance part="P+4" gate="VCC" x="254" y="187.96"/>
 <instance part="SUPPLY3" gate="GND" x="254" y="149.86"/>
-<instance part="SJ1" gate="G$1" x="109.22" y="187.96" smashed="yes" rot="R270">
-<attribute name="NAME" x="111.76" y="190.881" size="1.778" layer="95"/>
-<attribute name="VALUE" x="107.315" y="185.42" size="1.778" layer="96" rot="R270"/>
-</instance>
-<instance part="U$7" gate="A" x="99.06" y="101.6" rot="R180"/>
+<instance part="U$7" gate="A" x="101.6" y="101.6" rot="R180"/>
 <instance part="U$7" gate="B" x="101.6" y="78.74" rot="R180"/>
-<instance part="U$7" gate="C" x="175.26" y="38.1" rot="R180"/>
+<instance part="U$7" gate="C" x="198.12" y="38.1" rot="R180"/>
 <instance part="U$7" gate="D" x="198.12" y="7.62" rot="R180"/>
-<instance part="U$7" gate="E" x="274.32" y="127"/>
-<instance part="U$7" gate="F" x="124.46" y="127"/>
-<instance part="U$7" gate="PWR" x="284.48" y="27.94" rot="R180"/>
+<instance part="U$7" gate="E" x="261.62" y="78.74" rot="R180"/>
+<instance part="U$7" gate="F" x="261.62" y="106.68" rot="R180"/>
+<instance part="U$7" gate="PWR" x="353.06" y="48.26" rot="R180"/>
 </instances>
 <busses>
@@
 <nets>
 <net name="GND" class="0">
-<segment>
-<pinref part="U$34" gate="G$1" pin="1"/>
-<pinref part="SUPPLY1" gate="GND" pin="GND"/>
-<wire x1="76.2" y1="165.1" x2="68.58" y2="165.1" width="0.1524" layer="91"/>
-<wire x1="68.58" y1="165.1" x2="68.58" y2="162.56" width="0.1524" layer="91"/>
-</segment>
 <segment>
 <pinref part="U$31" gate="G$1" pin="VSSA"/>
@@
 <junction x="254" y="175.26"/>
 </segment>
-<segment>
-<pinref part="SJ1" gate="G$1" pin="2"/>
-<pinref part="P+2" gate="VCC" pin="VCC"/>
-<wire x1="109.22" y1="193.04" x2="109.22" y2="198.12" width="0.1524" layer="91"/>
-</segment>
 </net>
 <net name="MOSI_SI" class="0">
-<segment>
-<pinref part="U$34" gate="G$1" pin="4"/>
-<wire x1="91.44" y1="167.64" x2="109.22" y2="167.64" width="0.1524" layer="91"/>
-<label x="99.06" y="167.64" size="1.778" layer="95"/>
-</segment>
 <segment>
 <pinref part="U$31" gate="G$1" pin="SI"/>
@@
 <net name="SCLK" class="0">
 <segment>
-<pinref part="U$34" gate="G$1" pin="8"/>
-<wire x1="91.44" y1="172.72" x2="109.22" y2="172.72" width="0.1524" layer="91"/>
-<label x="99.06" y="172.72" size="1.778" layer="95"/>
-</segment>
-<segment>
 <pinref part="U$31" gate="G$1" pin="SCLK"/>
 <wire x1="279.4" y1="200.66" x2="259.08" y2="200.66" width="0.1524" layer="91"/>
@@
 <net name="CS" class="0">
 <segment>
-<pinref part="U$34" gate="G$1" pin="10"/>
-<wire x1="91.44" y1="175.26" x2="109.22" y2="175.26" width="0.1524" layer="91"/>
-<label x="99.06" y="175.26" size="1.778" layer="95"/>
-</segment>
-<segment>
 <pinref part="U$31" gate="G$1" pin="SCS"/>
 <wire x1="279.4" y1="190.5" x2="259.08" y2="190.5" width="0.1524" layer="91"/>
@@
 <label x="259.08" y="185.42" size="1.778" layer="95"/>
 </segment>
-<segment>
-<pinref part="U$34" gate="G$1" pin="7"/>
-<wire x1="76.2" y1="172.72" x2="60.96" y2="172.72" width="0.1524" layer="91"/>
-<label x="60.96" y="172.72" size="1.778" layer="95"/>
-</segment>
 </net>
 <net name="DISP_ENABLE" class="0">
-<segment>
-<pinref part="U$34" gate="G$1" pin="14"/>
-<wire x1="91.44" y1="180.34" x2="109.22" y2="180.34" width="0.1524" layer="91"/>
-<label x="99.06" y="180.34" size="1.778" layer="95"/>
-</segment>
 <segment>
 <pinref part="U$31" gate="G$1" pin="DISP"/>
@@
 <net name="EXTMODE" class="0">
 <segment>
-<pinref part="U$34" gate="G$1" pin="12"/>
-<wire x1="91.44" y1="177.8" x2="109.22" y2="177.8" width="0.1524" layer="91"/>
-<label x="99.06" y="177.8" size="1.778" layer="95"/>
-</segment>
-<segment>
 <pinref part="U$31" gate="G$1" pin="EXTMODE"/>
 <wire x1="279.4" y1="165.1" x2="259.08" y2="165.1" width="0.1524" layer="91"/>
@@
 </segment>
 </net>
-<net name="VMCU_3V3" class="0">
-<segment>
-<pinref part="U$34" gate="G$1" pin="2"/>
-<wire x1="116.84" y1="165.1" x2="91.44" y2="165.1" width="0.1524" layer="91"/>
-<wire x1="116.84" y1="165.1" x2="116.84" y2="187.96" width="0.1524" layer="91"/>
-<pinref part="SJ1" gate="G$1" pin="1"/>
-<wire x1="116.84" y1="187.96" x2="114.3" y2="187.96" width="0.1524" layer="91"/>
-<label x="99.06" y="165.1" size="1.778" layer="95"/>
-</segment>
-</net>
-<net name="5V" class="0">
-<segment>
-<pinref part="U$34" gate="G$1" pin="18"/>
-<wire x1="91.44" y1="185.42" x2="99.06" y2="185.42" width="0.1524" layer="91"/>
-<wire x1="99.06" y1="185.42" x2="99.06" y2="187.96" width="0.1524" layer="91"/>
-<pinref part="SJ1" gate="G$1" pin="3"/>
-<wire x1="99.06" y1="187.96" x2="104.14" y2="187.96" width="0.1524" layer="91"/>
-<label x="99.06" y="187.96" size="1.778" layer="95"/>
-</segment>
-</net>

Commit message: do cleanups, draw frame
Parts:
- removed C1, C2: 100nF, rcl:C-EUC0402K
- removed C3: 1uF, rcl:C-EUC0402K
- removed U$31: SHARP_MEM_LCD, sharp_mem_lcd:SHARP_MEM_LCD
- added JAD, JPOWER: (no value), SparkFun-Connectors:M06SIP
- added JEX: M08X2, SparkFun-Connectors:M08X2
- added JIOH, JIOL: (no value), SparkFun-Connectors:M081X08
Connections:
- removed net CS: U$31.SCS
- removed net DISP_ENABLE: C2.2, U$31.DISP
- removed net EXTCOMIN: U$31.EXTCOMIN
- removed net EXTMODE: U$31.EXTMODE
- removed net GND: C1.1, C2.1, C3.1, U$31.VSS, U$31.VSSA
- removed net MOSI_SI: U$31.SI
- removed net SCLK: U$31.SCLK
- removed net VCC: C1.2, C3.2, U$31.VDD, U$31.VDDA
- new net N$1: JIOH.1
- new net N$2: JAD.1
- new net N$3: JIOL.1
- new net N$4: JPOWER.1
Other:
- moved on the sheet: U$7PWR

Commit message: marching on
Parts:
- added C1, C2: (no value), maple-r5:CPOL-EUUD-4X5,8
- added C3: 0.1uF, SparkFun-Capacitors:0.1UF-25V-5%(0603)
- added PMIC1: MCP1700T-DIGITAL, maple-r5:MCP1700T
- added PMIC2: MCP1700T-ANALOG, maple-r5:MCP1700T
- added R1: 100, SparkFun-Resistors:100OHM1/10W1%(0603)
- added S1: SWITCH-MOMENTARY-2SMD, SparkFun-Electromechanical:SWITCH-MOMENTARY-2SMD
- added USB: PIXHAWK2_MOLEX-47346-0001, PX4FMUv1.7.1:PIXHAWK2_MOLEX-47346-0001
Connections:
- new net 3.3V: C1.+, PMIC1.VOUT
- new net GND: C1.-, C2.-, C3.1, PMIC1.GND, PMIC2.GND, R1.1, USB.5, USB.GND1, USB.GND2, USB.GND3
- new net N$5: C3.2, S1.2, U$7PWR.RESETN
- new net N$6: R1.2, S1.1
- new net VDD: C2.+, PMIC2.VOUT
Other:
- note removed: "Display"
- moved on the sheet: U$7E, U$7F
Changed lines of the file:
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@@
 <setting verticaltext="up"/>
 </settings>
-<grid distance="0.1" unitdist="inch" unit="inch" style="lines" multiple="1" display="yes" altdistance="0.01" altunitdist="inch" altunit="inch"/>
+<grid distance="0.05" unitdist="inch" unit="inch" style="lines" multiple="1" display="yes" altdistance="0.01" altunitdist="inch" altunit="inch"/>
 <layers>
 <layer number="1" name="Top" color="4" fill="1" visible="no" active="no"/>
@@
 <layer number="54" name="bGND_GNDA" color="1" fill="9" visible="no" active="no"/>
 <layer number="56" name="wert" color="7" fill="1" visible="no" active="no"/>
+<layer number="57" name="tCAD" color="7" fill="1" visible="no" active="no"/>
+<layer number="58" name="bCAD" color="7" fill="1" visible="no" active="no"/>
 <layer number="91" name="Nets" color="2" fill="1" visible="yes" active="yes"/>
 <layer number="92" name="Busses" color="1" fill="1" visible="yes" active="yes"/>
@@
 <layer number="108" name="tplace-old" color="10" fill="1" visible="yes" active="yes"/>
 <layer number="109" name="ref-old" color="11" fill="1" visible="yes" active="yes"/>
+<layer number="110" name="fp0" color="7" fill="1" visible="yes" active="yes"/>
 <layer number="116" name="Patch_BOT" color="9" fill="4" visible="no" active="yes"/>
 <layer number="121" name="_tsilk" color="7" fill="1" visible="no" active="yes"/>
 <layer number="122" name="_bsilk" color="7" fill="1" visible="no" active="yes"/>
+<layer number="123" name="tTestmark" color="7" fill="1" visible="yes" active="yes"/>
+<layer number="124" name="bTestmark" color="7" fill="1" visible="yes" active="yes"/>
 <layer number="125" name="_tNames" color="7" fill="1" visible="yes" active="yes"/>
+<layer number="131" name="tAdjust" color="7" fill="1" visible="yes" active="yes"/>
+<layer number="132" name="bAdjust" color="7" fill="1" visible="yes" active="yes"/>
 <layer number="144" name="Drill_legend" color="7" fill="1" visible="yes" active="yes"/>
 <layer number="151" name="HeatSink" color="7" fill="1" visible="no" active="yes"/>
@@
 <part name="JEX" library="SparkFun-Connectors" deviceset="M08X2" device=""/>
 <part name="FRAME1" library="SparkFun-Aesthetics" deviceset="FRAME-A3" device=""/>
+<part name="PMIC1" library="maple-r5" deviceset="MCP1700T" device="" value="MCP1700T-DIGITAL"/>
+<part name="PMIC2" library="maple-r5" deviceset="MCP1700T" device="" value="MCP1700T-ANALOG"/>
+<part name="C1" library="maple-r5" deviceset="CPOL-EU" device="UD-4X5,8"/>
+<part name="C2" library="maple-r5" deviceset="CPOL-EU" device="UD-4X5,8"/>
+<part name="SUPPLY1" library="SparkFun-Aesthetics" deviceset="3.3V" device=""/>
+<part name="GND2" library="SparkFun-Aesthetics" deviceset="GND" device=""/>
+<part name="VDDA" library="maple-r5" deviceset="VDD" device=""/>
+<part name="GND1" library="SparkFun-Aesthetics" deviceset="GND" device=""/>
+<part name="S1" library="SparkFun-Electromechanical" deviceset="SWITCH-MOMENTARY-2" device="SMD"/>
+<part name="R1" library="SparkFun-Resistors" deviceset="100OHM1/10W1%(0603)" device="" value="100"/>
+<part name="C3" library="SparkFun-Capacitors" deviceset="0.1UF-25V-5%(0603)" device="" value="0.1uF"/>
+<part name="GND3" library="SparkFun-Aesthetics" deviceset="GND" device=""/>
+<part name="USB" library="PX4FMUv1.7.1" deviceset="PIXHAWK2_MOLEX-47346-0001" device=""/>
+<part name="GND4" library="SparkFun-Aesthetics" deviceset="GND" device=""/>
 </parts>
 <sheets>
@@
 <wire x1="144.78" y1="134.62" x2="144.78" y2="256.54" width="0.1524" layer="97" style="shortdash"/>
 <text x="15.24" y="241.3" size="3.81" layer="97">Expansion Header Connector</text>
-<text x="205.74" y="243.84" size="3.81" layer="97">Display</text>
-<text x="344.17" y="20.574" size="2.54" layer="94" font="vector">Librae</text>
+<text x="330.2" y="4.318" size="2.54" layer="94" font="vector">Librae</text>
 <wire x1="5.08" y1="134.62" x2="144.78" y2="134.62" width="0.1524" layer="97"/>
 <wire x1="144.78" y1="134.62" x2="381" y2="134.62" width="0.1524" layer="97"/>
@@
 <instance part="U$7" gate="C" x="198.12" y="38.1" rot="R180"/>
 <instance part="U$7" gate="D" x="198.12" y="7.62" rot="R180"/>
-<instance part="U$7" gate="E" x="261.62" y="78.74" rot="R180"/>
-<instance part="U$7" gate="F" x="261.62" y="106.68" rot="R180"/>
+<instance part="U$7" gate="E" x="226.06" y="101.6" rot="R180"/>
+<instance part="U$7" gate="F" x="243.84" y="78.74" rot="R180"/>
 <instance part="U$7" gate="PWR" x="347.98" y="53.34" rot="R180"/>
 <instance part="JIOH" gate="G$1" x="27.94" y="220.98"/>
@@
 <instance part="JEX" gate="G$1" x="104.14" y="223.52" rot="R180"/>
 <instance part="FRAME1" gate="G$1" x="0" y="0"/>
+<instance part="PMIC1" gate="G$1" x="347.98" y="215.9" rot="MR0"/>
+<instance part="PMIC2" gate="G$1" x="287.02" y="215.9"/>
+<instance part="C1" gate="G$1" x="330.2" y="215.9" rot="MR0"/>
+<instance part="C2" gate="G$1" x="304.8" y="215.9"/>
+<instance part="SUPPLY1" gate="G$1" x="330.2" y="223.52" rot="MR0"/>
+<instance part="GND2" gate="1" x="330.2" y="205.74"/>
+<instance part="VDDA" gate="G$1" x="304.8" y="226.06"/>
+<instance part="GND1" gate="1" x="304.8" y="205.74" rot="MR0"/>
+<instance part="S1" gate="G$1" x="340.36" y="45.72"/>
+<instance part="R1" gate="G$1" x="330.2" y="40.64" rot="R90"/>
+<instance part="C3" gate="G$1" x="347.98" y="40.64" rot="R180"/>
+<instance part="GND3" gate="1" x="347.98" y="27.94"/>
+<instance part="USB" gate="G$1" x="271.78" y="111.76" rot="R90"/>
+<instance part="GND4" gate="1" x="287.02" y="99.06"/>
 </instances>
 <busses>
@@
 </segment>
 </net>
+<net name="3.3V" class="0">
+<segment>
+<pinref part="PMIC1" gate="G$1" pin="VOUT"/>
+<wire x1="337.82" y1="220.98" x2="330.2" y2="220.98" width="0.1524" layer="91"/>
+<pinref part="C1" gate="G$1" pin="+"/>
+<wire x1="330.2" y1="220.98" x2="330.2" y2="218.44" width="0.1524" layer="91"/>
+<pinref part="SUPPLY1" gate="G$1" pin="3.3V"/>
+<wire x1="330.2" y1="223.52" x2="330.2" y2="220.98" width="0.1524" layer="91"/>
+<junction x="330.2" y="220.98"/>
+</segment>
+</net>
+<net name="VDD" class="0">
+<segment>
+<pinref part="PMIC2" gate="G$1" pin="VOUT"/>
+<wire x1="297.18" y1="220.98" x2="304.8" y2="220.98" width="0.1524" layer="91"/>
+<pinref part="C2" gate="G$1" pin="+"/>
+<wire x1="304.8" y1="220.98" x2="304.8" y2="218.44" width="0.1524" layer="91"/>
+<wire x1="304.8" y1="223.52" x2="304.8" y2="220.98" width="0.1524" layer="91"/>
+<pinref part="VDDA" gate="G$1" pin="VDD"/>
+<junction x="304.8" y="220.98"/>
+</segment>
+</net>
+<net name="GND" class="0">
+<segment>
+<pinref part="C1" gate="G$1" pin="-"/>
+<junction x="330.2" y="210.82"/>
+<pinref part="PMIC1" gate="G$1" pin="GND"/>
+<wire x1="337.82" y1="210.82" x2="330.2" y2="210.82" width="0.1524" layer="91"/>
+<pinref part="GND2" gate="1" pin="GND"/>
+<wire x1="330.2" y1="210.82" x2="330.2" y2="208.28" width="0.1524" layer="91"/>
+</segment>
+<segment>
+<pinref part="PMIC2" gate="G$1" pin="GND"/>
+<pinref part="C2" gate="G$1" pin="-"/>
+<wire x1="297.18" y1="210.82" x2="304.8" y2="210.82" width="0.1524" layer="91"/>
+<pinref part="GND1" gate="1" pin="GND"/>
+<wire x1="304.8" y1="210.82" x2="304.8" y2="208.28" width="0.1524" layer="91"/>
+<junction x="304.8" y="210.82"/>
+</segment>
+<segment>
+<pinref part="R1" gate="G$1" pin="1"/>
+<wire x1="330.2" y1="35.56" x2="330.2" y2="33.02" width="0.1524" layer="91"/>
+<wire x1="330.2" y1="33.02" x2="347.98" y2="33.02" width="0.1524" layer="91"/>
+<pinref part="GND3" gate="1" pin="GND"/>
+<wire x1="347.98" y1="30.48" x2="347.98" y2="33.02" width="0.1524" layer="91"/>
+<pinref part="C3" gate="G$1" pin="1"/>
+<wire x1="347.98" y1="33.02" x2="347.98" y2="35.56" width="0.1524" layer="91"/>
+<junction x="347.98" y="33.02"/>
+</segment>
+<segment>
+<pinref part="USB" gate="G$1" pin="5"/>
+<wire x1="276.86" y1="106.68" x2="276.86" y2="104.14" width="0.1524" layer="91"/>
+<wire x1="284.48" y1="118.11" x2="287.02" y2="118.11" width="0.1524" layer="91"/>
+<pinref part="GND4" gate="1" pin="GND"/>
+<wire x1="287.02" y1="118.11" x2="287.02" y2="115.57" width="0.1524" layer="91"/>
+<wire x1="287.02" y1="115.57" x2="287.02" y2="113.03" width="0.1524" layer="91"/>
+<wire x1="287.02" y1="113.03" x2="287.02" y2="110.49" width="0.1524" layer="91"/>
+<wire x1="287.02" y1="110.49" x2="287.02" y2="104.14" width="0.1524" layer="91"/>
+<wire x1="287.02" y1="104.14" x2="287.02" y2="101.6" width="0.1524" layer="91"/>
+<wire x1="276.86" y1="104.14" x2="287.02" y2="104.14" width="0.1524" layer="91"/>
+<pinref part="USB" gate="G$1" pin="GND1"/>
+<wire x1="284.48" y1="110.49" x2="287.02" y2="110.49" width="0.1524" layer="91"/>
+<pinref part="USB" gate="G$1" pin="GND2"/>
+<wire x1="284.48" y1="113.03" x2="287.02" y2="113.03" width="0.1524" layer="91"/>
+<pinref part="USB" gate="G$1" pin="GND3"/>
+<wire x1="284.48" y1="115.57" x2="287.02" y2="115.57" width="0.1524" layer="91"/>
+<junction x="287.02" y="115.57"/>
+<junction x="287.02" y="113.03"/>
+<junction x="287.02" y="110.49"/>
+<junction x="287.02" y="104.14"/>
+</segment>
+</net>
+<net name="N$5" class="0">
+<segment>
+<pinref part="U$7" gate="PWR" pin="RESETN"/>
+<wire x1="347.98" y1="55.88" x2="347.98" y2="45.72" width="0.1524" layer="91"/>
+<pinref part="S1" gate="G$1" pin="2"/>
+<wire x1="347.98" y1="45.72" x2="345.44" y2="45.72" width="0.1524" layer="91"/>
+<pinref part="C3" gate="G$1" pin="2"/>
+<wire x1="347.98" y1="43.18" x2="347.98" y2="45.72" width="0.1524" layer="91"/>
+<junction x="347.98" y="45.72"/>
+</segment>
+</net>
+<net name="N$6" class="0">
+<segment>
+<pinref part="S1" gate="G$1" pin="1"/>
+<pinref part="R1" gate="G$1" pin="2"/>
+<wire x1="335.28" y1="45.72" x2="330.2" y2="45.72" width="0.1524" layer="91"/>
+</segment>
+</net>
