File: efm32core.sch (EAGLE design)
At the start: 66 parts, among them Q1 MMBT5088, U3 USD-SOCKETNEW, X1 48.0MHz, Y1 32.768kHz

Commit message: route
Connections:
- removed net VIN: JPOWER.6
- new net N$5: U3.SHIELD@2
- net 5V: now also JPOWER.6
- net GND: now also JIOH.7, U3.SHIELD@1, U3.SHIELD@3, U3.SHIELD@4
- net US1_RX: now also BLE112-A.P0_3
- net US1_TX: now also BLE112-A.P0_2
Changed lines of the file:
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@@
 <setting verticaltext="up"/>
 </settings>
-<grid distance="0.1" unitdist="inch" unit="inch" style="lines" multiple="1" display="no" altdistance="0.01" altunitdist="inch" altunit="inch"/>
+<grid distance="0.1" unitdist="inch" unit="inch" style="lines" multiple="1" display="yes" altdistance="0.01" altunitdist="inch" altunit="inch"/>
 <layers>
 <layer number="1" name="Top" color="4" fill="1" visible="no" active="no"/>
@@
 <part name="SJ2" library="BLE112-Breakout-Board-v2.1" deviceset="JUMPER_SJ" device=""/>
 <part name="R10" library="SparkFun-Resistors" deviceset="100-1%" device="" value="1.5k"/>
+<part name="GND23" library="SparkFun-Aesthetics" deviceset="GND" device=""/>
+<part name="GND24" library="SparkFun-Aesthetics" deviceset="GND" device=""/>
 </parts>
 <sheets>
@@
 <instance part="SJ2" gate="1" x="139.7" y="238.76"/>
 <instance part="R10" gate="G$1" x="144.78" y="210.82" rot="R90"/>
+<instance part="GND23" gate="1" x="43.18" y="228.6" rot="R90"/>
+<instance part="GND24" gate="1" x="226.06" y="231.14" rot="R90"/>
 </instances>
 <busses>
@@
 <wire x1="226.06" y1="165.1" x2="226.06" y2="167.64" width="0.1524" layer="91"/>
 </segment>
+<segment>
+<pinref part="JIOH" gate="G$1" pin="7"/>
+<wire x1="33.02" y1="228.6" x2="40.64" y2="228.6" width="0.1524" layer="91"/>
+<pinref part="GND23" gate="1" pin="GND"/>
+</segment>
+<segment>
+<pinref part="U3" gate="G$1" pin="SHIELD@1"/>
+<wire x1="215.9" y1="231.14" x2="220.98" y2="231.14" width="0.1524" layer="91"/>
+<pinref part="GND24" gate="1" pin="GND"/>
+<pinref part="U3" gate="G$1" pin="SHIELD@4"/>
+<wire x1="220.98" y1="231.14" x2="223.52" y2="231.14" width="0.1524" layer="91"/>
+<wire x1="215.9" y1="238.76" x2="220.98" y2="238.76" width="0.1524" layer="91"/>
+<wire x1="220.98" y1="238.76" x2="220.98" y2="236.22" width="0.1524" layer="91"/>
+<junction x="220.98" y="231.14"/>
+<pinref part="U3" gate="G$1" pin="SHIELD@3"/>
+<wire x1="220.98" y1="236.22" x2="220.98" y2="233.68" width="0.1524" layer="91"/>
+<wire x1="220.98" y1="233.68" x2="220.98" y2="231.14" width="0.1524" layer="91"/>
+<wire x1="215.9" y1="236.22" x2="220.98" y2="236.22" width="0.1524" layer="91"/>
+<junction x="220.98" y="236.22"/>
+<wire x1="220.98" y1="233.68" x2="223.52" y2="233.68" width="0.1524" layer="91"/>
+</segment>
 </net>
 <net name="5V" class="0">
@@
 <junction x="358.14" y="190.5"/>
 </segment>
+<segment>
+<pinref part="JPOWER" gate="G$1" pin="6"/>
+<wire x1="78.74" y1="200.66" x2="86.36" y2="200.66" width="0.1524" layer="91"/>
+<label x="81.28" y="200.66" size="1.778" layer="95"/>
+</segment>
 </net>
 <net name="RESET" class="0">
@@
 </segment>
 </net>
-<net name="VIN" class="0">
-<segment>
-<pinref part="JPOWER" gate="G$1" pin="6"/>
-<wire x1="78.74" y1="200.66" x2="86.36" y2="200.66" width="0.1524" layer="91"/>
-<label x="81.28" y="200.66" size="1.778" layer="95"/>
-</segment>
-</net>
 <net name="ADCH0" class="0">
 <segment>
@@
 <label x="200.66" y="7.62" size="1.778" layer="95"/>
 </segment>
+<segment>
+<pinref part="BLE112-A" gate="G$1" pin="P0_2"/>
+<wire x1="213.36" y1="170.18" x2="220.98" y2="170.18" width="0.1524" layer="91"/>
+<label x="213.36" y="170.18" size="1.778" layer="95"/>
+</segment>
 </net>
 <net name="US1_RX" class="0">
@@
 <wire x1="198.12" y1="10.16" x2="205.74" y2="10.16" width="0.1524" layer="91"/>
 <label x="200.66" y="10.16" size="1.778" layer="95"/>
+</segment>
+<segment>
+<pinref part="BLE112-A" gate="G$1" pin="P0_3"/>
+<wire x1="213.36" y1="167.64" x2="220.98" y2="167.64" width="0.1524" layer="91"/>
+<label x="213.36" y="167.64" size="1.778" layer="95"/>
 </segment>
 </net>
@@
 </segment>
 </net>
+<net name="N$5" class="0">
+<segment>
+<pinref part="U3" gate="G$1" pin="SHIELD@2"/>
+<wire x1="215.9" y1="233.68" x2="220.98" y2="233.68" width="0.1524" layer="91"/>
+<label x="218.44" y="233.68" size="1.778" layer="95"/>
+</segment>
+</net>

Commit message: layout and refine wires
Connections:
- removed net N$1: JIOH.1
- removed net N$20: R11.1
- removed net PD6: MCUD.PD6/ACMP0_O#2/ADC0_CH6/DAC0_P1/OPAMP_P1/ETM_TD0#0/I2C0_SDA#1/LES_ALTEX0/LETIM0_OUT0#0/PCNT0_S0IN#3/TIM1_CC0#4/US1_RX#2
- removed net PD7: MCUD.PD7/ACMP1_O#2/ADC0_CH7/CMU_CLK0#2/DAC0_N1/OPAMP_N1/ETM_TCLK#0/I2C0_SCL#1/LES_ALTEX1/LETIM0_OUT1#0/PCNT0_S1IN#3/TIM1_CC1#4/US1_TX#2
- new net IO10: MCUA.PA5/ETM_TD3#3/LES_ALTEX4/LEU1_TX#1/TIM0_CDTI2#0, R11.1
- new net IO8: JIOH.1, MCUA.PA3/ETM_TD1#3/LES_ALTEX2/TIM0_CDTI0#0
- new net IO9: JIOH.2, MCUA.PA4/ETM_TD2#3/LES_ALTEX3/TIM0_CDTI1#0
- new net US1_CLK_2: JIOH.6, MCUF.PF0/DBG_SWCLK#0,1,2,3/I2C0_SDA#5/LETIM0_OUT0#2/LEU0_TX#3/TIM0_CC0#5/US1_CLK#2
- new net US1_CS_2: JIOH.3, MCUF.PF1/DBG_SWDIO#0,1,2,3/GPIO_EM4WU3/I2C0_SCL#5/LETIM0_OUT1#2/LEU0_RX#3/TIM0_CC1#5/US1_CS#2
- new net US1_RX_2: JIOH.5, MCUD.PD6/ACMP0_O#2/ADC0_CH6/DAC0_P1/OPAMP_P1/ETM_TD0#0/I2C0_SDA#1/LES_ALTEX0/LETIM0_OUT0#0/PCNT0_S0IN#3/TIM1_CC0#4/US1_RX#2
- new net US1_TX_2: JIOH.4, MCUD.PD7/ACMP1_O#2/ADC0_CH7/CMU_CLK0#2/DAC0_N1/OPAMP_N1/ETM_TCLK#0/I2C0_SCL#1/LES_ALTEX1/LETIM0_OUT1#0/PCNT0_S1IN#3/TIM1_CC1#4/US1_TX#2
Changed lines of the file:
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@@
 <instance part="SJ2" gate="1" x="139.7" y="238.76"/>
 <instance part="R10" gate="G$1" x="144.78" y="210.82" rot="R90"/>
-<instance part="GND23" gate="1" x="43.18" y="228.6" rot="R90"/>
+<instance part="GND23" gate="1" x="50.8" y="228.6" rot="R90"/>
 <instance part="GND24" gate="1" x="226.06" y="231.14" rot="R90"/>
 </instances>
@@
 </busses>
 <nets>
-<net name="N$1" class="0">
-<segment>
-<pinref part="JIOH" gate="G$1" pin="1"/>
-<wire x1="33.02" y1="213.36" x2="40.64" y2="213.36" width="0.1524" layer="91"/>
-</segment>
-</net>
 <net name="N$3" class="0">
 <segment>
@@
 <segment>
 <pinref part="JIOH" gate="G$1" pin="7"/>
-<wire x1="33.02" y1="228.6" x2="40.64" y2="228.6" width="0.1524" layer="91"/>
+<wire x1="33.02" y1="228.6" x2="48.26" y2="228.6" width="0.1524" layer="91"/>
 <pinref part="GND23" gate="1" pin="GND"/>
 </segment>
@@
 <wire x1="33.02" y1="165.1" x2="40.64" y2="165.1" width="0.1524" layer="91"/>
 <label x="35.56" y="165.1" size="1.778" layer="95"/>
-</segment>
-</net>
-<net name="PD6" class="0">
-<segment>
-<pinref part="MCU" gate="D" pin="PD6/ACMP0_O#2/ADC0_CH6/DAC0_P1/OPAMP_P1/ETM_TD0#0/I2C0_SDA#1/LES_ALTEX0/LETIM0_OUT0#0/PCNT0_S0IN#3/TIM1_CC0#4/US1_RX#2"/>
-<wire x1="198.12" y1="60.96" x2="205.74" y2="60.96" width="0.1524" layer="91"/>
-<label x="200.66" y="60.96" size="1.778" layer="95"/>
-</segment>
-</net>
-<net name="PD7" class="0">
-<segment>
-<pinref part="MCU" gate="D" pin="PD7/ACMP1_O#2/ADC0_CH7/CMU_CLK0#2/DAC0_N1/OPAMP_N1/ETM_TCLK#0/I2C0_SCL#1/LES_ALTEX1/LETIM0_OUT1#0/PCNT0_S1IN#3/TIM1_CC1#4/US1_TX#2"/>
-<wire x1="198.12" y1="63.5" x2="205.74" y2="63.5" width="0.1524" layer="91"/>
-<label x="200.66" y="63.5" size="1.778" layer="95"/>
 </segment>
 </net>
@@
 </segment>
 </net>
-<net name="N$20" class="0">
-<segment>
-<pinref part="R11" gate="G$1" pin="1"/>
-<wire x1="137.16" y1="175.26" x2="132.08" y2="175.26" width="0.1524" layer="91"/>
-<label x="129.54" y="175.26" size="1.778" layer="95"/>
-<label x="129.54" y="175.26" size="1.778" layer="95"/>
-</segment>
-</net>
 <net name="BLE-RST" class="0">
 <segment>
@@
 </segment>
 </net>
+<net name="IO10" class="0">
+<segment>
+<pinref part="MCU" gate="A" pin="PA5/ETM_TD3#3/LES_ALTEX4/LEU1_TX#1/TIM0_CDTI2#0"/>
+<wire x1="101.6" y1="116.84" x2="109.22" y2="116.84" width="0.1524" layer="91"/>
+<label x="104.14" y="116.84" size="1.778" layer="95"/>
+</segment>
+<segment>
+<pinref part="R11" gate="G$1" pin="1"/>
+<wire x1="137.16" y1="175.26" x2="132.08" y2="175.26" width="0.1524" layer="91"/>
+<label x="129.54" y="175.26" size="1.778" layer="95"/>
+</segment>
+</net>
+<net name="US1_CLK_2" class="0">
+<segment>
+<pinref part="JIOH" gate="G$1" pin="6"/>
+<wire x1="33.02" y1="226.06" x2="40.64" y2="226.06" width="0.1524" layer="91"/>
+<label x="35.56" y="226.06" size="1.778" layer="95"/>
+</segment>
+<segment>
+<pinref part="MCU" gate="F" pin="PF0/DBG_SWCLK#0,1,2,3/I2C0_SDA#5/LETIM0_OUT0#2/LEU0_TX#3/TIM0_CC0#5/US1_CLK#2"/>
+<wire x1="241.3" y1="109.22" x2="248.92" y2="109.22" width="0.1524" layer="91"/>
+<label x="243.84" y="109.22" size="1.778" layer="95"/>
+</segment>
+</net>
+<net name="IO8" class="0">
+<segment>
+<pinref part="MCU" gate="A" pin="PA3/ETM_TD1#3/LES_ALTEX2/TIM0_CDTI0#0"/>
+<wire x1="101.6" y1="111.76" x2="109.22" y2="111.76" width="0.1524" layer="91"/>
+<label x="104.14" y="111.76" size="1.778" layer="95"/>
+</segment>
+<segment>
+<pinref part="JIOH" gate="G$1" pin="1"/>
+<wire x1="33.02" y1="213.36" x2="40.64" y2="213.36" width="0.1524" layer="91"/>
+<label x="35.56" y="213.36" size="1.778" layer="95"/>
+</segment>
+</net>
+<net name="IO9" class="0">
+<segment>
+<pinref part="MCU" gate="A" pin="PA4/ETM_TD2#3/LES_ALTEX3/TIM0_CDTI1#0"/>
+<wire x1="101.6" y1="114.3" x2="109.22" y2="114.3" width="0.1524" layer="91"/>
+<label x="104.14" y="114.3" size="1.778" layer="95"/>
+</segment>
+<segment>
+<pinref part="JIOH" gate="G$1" pin="2"/>
+<wire x1="33.02" y1="215.9" x2="40.64" y2="215.9" width="0.1524" layer="91"/>
+<label x="35.56" y="215.9" size="1.778" layer="95"/>
+</segment>
+</net>
+<net name="US1_RX_2" class="0">
+<segment>
+<pinref part="JIOH" gate="G$1" pin="5"/>
+<wire x1="33.02" y1="223.52" x2="40.64" y2="223.52" width="0.1524" layer="91"/>
+<label x="35.56" y="223.52" size="1.778" layer="95"/>
+</segment>
+<segment>
+<pinref part="MCU" gate="D" pin="PD6/ACMP0_O#2/ADC0_CH6/DAC0_P1/OPAMP_P1/ETM_TD0#0/I2C0_SDA#1/LES_ALTEX0/LETIM0_OUT0#0/PCNT0_S0IN#3/TIM1_CC0#4/US1_RX#2"/>
+<wire x1="198.12" y1="60.96" x2="205.74" y2="60.96" width="0.1524" layer="91"/>
+<label x="200.66" y="60.96" size="1.778" layer="95"/>
+</segment>
+</net>
+<net name="US1_TX_2" class="0">
+<segment>
+<pinref part="JIOH" gate="G$1" pin="4"/>
+<wire x1="33.02" y1="220.98" x2="40.64" y2="220.98" width="0.1524" layer="91"/>
+<label x="35.56" y="220.98" size="1.778" layer="95"/>
+</segment>
+<segment>
+<pinref part="MCU" gate="D" pin="PD7/ACMP1_O#2/ADC0_CH7/CMU_CLK0#2/DAC0_N1/OPAMP_N1/ETM_TCLK#0/I2C0_SCL#1/LES_ALTEX1/LETIM0_OUT1#0/PCNT0_S1IN#3/TIM1_CC1#4/US1_TX#2"/>
+<wire x1="198.12" y1="63.5" x2="205.74" y2="63.5" width="0.1524" layer="91"/>
+<label x="200.66" y="63.5" size="1.778" layer="95"/>
+</segment>
+</net>
+<net name="US1_CS_2" class="0">
+<segment>
+<pinref part="JIOH" gate="G$1" pin="3"/>
+<wire x1="33.02" y1="218.44" x2="40.64" y2="218.44" width="0.1524" layer="91"/>
+<label x="35.56" y="218.44" size="1.778" layer="95"/>
+</segment>
+<segment>
+<pinref part="MCU" gate="F" pin="PF1/DBG_SWDIO#0,1,2,3/GPIO_EM4WU3/I2C0_SCL#5/LETIM0_OUT1#2/LEU0_RX#3/TIM0_CC1#5/US1_CS#2"/>
+<wire x1="241.3" y1="111.76" x2="248.92" y2="111.76" width="0.1524" layer="91"/>
+<label x="243.84" y="111.76" size="1.778" layer="95"/>
+</segment>
+</net>

Commit message: some refines
Connections:
- removed net US1_CLK_2: JIOH.6, MCUF.PF0/DBG_SWCLK#0,1,2,3/I2C0_SDA#5/LETIM0_OUT0#2/LEU0_TX#3/TIM0_CC0#5/US1_CLK#2
- removed net US1_CS_2: JIOH.3, MCUF.PF1/DBG_SWDIO#0,1,2,3/GPIO_EM4WU3/I2C0_SCL#5/LETIM0_OUT1#2/LEU0_RX#3/TIM0_CC1#5/US1_CS#2
- removed net US1_RX_2: JIOH.5, MCUD.PD6/ACMP0_O#2/ADC0_CH6/DAC0_P1/OPAMP_P1/ETM_TD0#0/I2C0_SDA#1/LES_ALTEX0/LETIM0_OUT0#0/PCNT0_S0IN#3/TIM1_CC0#4/US1_RX#2
- removed net US1_TX_2: JIOH.4, MCUD.PD7/ACMP1_O#2/ADC0_CH7/CMU_CLK0#2/DAC0_N1/OPAMP_N1/ETM_TCLK#0/I2C0_SCL#1/LES_ALTEX1/LETIM0_OUT1#0/PCNT0_S1IN#3/TIM1_CC1#4/US1_TX#2
- new net US0_CLK: JIOH.6, MCUE.PE12/CMU_CLK1#2/I2C0_SDA#6/LES_ALTEX6/TIM1_CC2#1/US0_CLK#0/US0_RX#3
- new net US0_CS: JIOH.3, MCUE.PE13/ACMP0_O#0/GPIO_EM4WU5/I2C0_SCL#6/LES_ALTEX7/US0_CS#0/US0_TX#3
- net US0_RX: now also JIOH.5
- net US0_TX: now also JIOH.4
Changed lines of the file:
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@@
 <label x="243.84" y="83.82" size="1.778" layer="95"/>
+</segment>
+<segment>
+<pinref part="JIOH" gate="G$1" pin="4"/>
+<wire x1="33.02" y1="220.98" x2="40.64" y2="220.98" width="0.1524" layer="91"/>
+<label x="35.56" y="220.98" size="1.778" layer="95"/>
 </segment>
 </net>
@@
 <wire x1="241.3" y1="86.36" x2="248.92" y2="86.36" width="0.1524" layer="91"/>
 <label x="243.84" y="86.36" size="1.778" layer="95"/>
+</segment>
+<segment>
+<pinref part="JIOH" gate="G$1" pin="5"/>
+<wire x1="33.02" y1="223.52" x2="40.64" y2="223.52" width="0.1524" layer="91"/>
+<label x="35.56" y="223.52" size="1.778" layer="95"/>
 </segment>
 </net>
@@
 </segment>
 </net>
-<net name="US1_CLK_2" class="0">
+<net name="IO8" class="0">
+<segment>
+<pinref part="MCU" gate="A" pin="PA3/ETM_TD1#3/LES_ALTEX2/TIM0_CDTI0#0"/>
+<wire x1="101.6" y1="111.76" x2="109.22" y2="111.76" width="0.1524" layer="91"/>
+<label x="104.14" y="111.76" size="1.778" layer="95"/>
+</segment>
+<segment>
+<pinref part="JIOH" gate="G$1" pin="1"/>
+<wire x1="33.02" y1="213.36" x2="40.64" y2="213.36" width="0.1524" layer="91"/>
+<label x="35.56" y="213.36" size="1.778" layer="95"/>
+</segment>
+</net>
+<net name="IO9" class="0">
+<segment>
+<pinref part="MCU" gate="A" pin="PA4/ETM_TD2#3/LES_ALTEX3/TIM0_CDTI1#0"/>
+<wire x1="101.6" y1="114.3" x2="109.22" y2="114.3" width="0.1524" layer="91"/>
+<label x="104.14" y="114.3" size="1.778" layer="95"/>
+</segment>
+<segment>
+<pinref part="JIOH" gate="G$1" pin="2"/>
+<wire x1="33.02" y1="215.9" x2="40.64" y2="215.9" width="0.1524" layer="91"/>
+<label x="35.56" y="215.9" size="1.778" layer="95"/>
+</segment>
+</net>
+<net name="US0_CLK" class="0">
+<segment>
+<pinref part="MCU" gate="E" pin="PE12/CMU_CLK1#2/I2C0_SDA#6/LES_ALTEX6/TIM1_CC2#1/US0_CLK#0/US0_RX#3"/>
+<wire x1="241.3" y1="88.9" x2="248.92" y2="88.9" width="0.1524" layer="91"/>
+<label x="243.84" y="88.9" size="1.778" layer="95"/>
+</segment>
 <segment>
 <pinref part="JIOH" gate="G$1" pin="6"/>
@@
 <label x="35.56" y="226.06" size="1.778" layer="95"/>
 </segment>
-<segment>
-<pinref part="MCU" gate="F" pin="PF0/DBG_SWCLK#0,1,2,3/I2C0_SDA#5/LETIM0_OUT0#2/LEU0_TX#3/TIM0_CC0#5/US1_CLK#2"/>
-<wire x1="241.3" y1="109.22" x2="248.92" y2="109.22" width="0.1524" layer="91"/>
-<label x="243.84" y="109.22" size="1.778" layer="95"/>
-</segment>
-</net>
-<net name="IO8" class="0">
-<segment>
-<pinref part="MCU" gate="A" pin="PA3/ETM_TD1#3/LES_ALTEX2/TIM0_CDTI0#0"/>
-<wire x1="101.6" y1="111.76" x2="109.22" y2="111.76" width="0.1524" layer="91"/>
-<label x="104.14" y="111.76" size="1.778" layer="95"/>
-</segment>
-<segment>
-<pinref part="JIOH" gate="G$1" pin="1"/>
-<wire x1="33.02" y1="213.36" x2="40.64" y2="213.36" width="0.1524" layer="91"/>
-<label x="35.56" y="213.36" size="1.778" layer="95"/>
-</segment>
-</net>
-<net name="IO9" class="0">
-<segment>
-<pinref part="MCU" gate="A" pin="PA4/ETM_TD2#3/LES_ALTEX3/TIM0_CDTI1#0"/>
-<wire x1="101.6" y1="114.3" x2="109.22" y2="114.3" width="0.1524" layer="91"/>
-<label x="104.14" y="114.3" size="1.778" layer="95"/>
-</segment>
-<segment>
-<pinref part="JIOH" gate="G$1" pin="2"/>
-<wire x1="33.02" y1="215.9" x2="40.64" y2="215.9" width="0.1524" layer="91"/>
-<label x="35.56" y="215.9" size="1.778" layer="95"/>
-</segment>
-</net>
-<net name="US1_RX_2" class="0">
-<segment>
-<pinref part="JIOH" gate="G$1" pin="5"/>
-<wire x1="33.02" y1="223.52" x2="40.64" y2="223.52" width="0.1524" layer="91"/>
-<label x="35.56" y="223.52" size="1.778" layer="95"/>
-</segment>
-<segment>
-<pinref part="MCU" gate="D" pin="PD6/ACMP0_O#2/ADC0_CH6/DAC0_P1/OPAMP_P1/ETM_TD0#0/I2C0_SDA#1/LES_ALTEX0/LETIM0_OUT0#0/PCNT0_S0IN#3/TIM1_CC0#4/US1_RX#2"/>
-<wire x1="198.12" y1="60.96" x2="205.74" y2="60.96" width="0.1524" layer="91"/>
-<label x="200.66" y="60.96" size="1.778" layer="95"/>
-</segment>
-</net>
-<net name="US1_TX_2" class="0">
-<segment>
-<pinref part="JIOH" gate="G$1" pin="4"/>
-<wire x1="33.02" y1="220.98" x2="40.64" y2="220.98" width="0.1524" layer="91"/>
-<label x="35.56" y="220.98" size="1.778" layer="95"/>
-</segment>
-<segment>
-<pinref part="MCU" gate="D" pin="PD7/ACMP1_O#2/ADC0_CH7/CMU_CLK0#2/DAC0_N1/OPAMP_N1/ETM_TCLK#0/I2C0_SCL#1/LES_ALTEX1/LETIM0_OUT1#0/PCNT0_S1IN#3/TIM1_CC1#4/US1_TX#2"/>
-<wire x1="198.12" y1="63.5" x2="205.74" y2="63.5" width="0.1524" layer="91"/>
-<label x="200.66" y="63.5" size="1.778" layer="95"/>
-</segment>
-</net>
-<net name="US1_CS_2" class="0">
+</net>
+<net name="US0_CS" class="0">
+<segment>
+<pinref part="MCU" gate="E" pin="PE13/ACMP0_O#0/GPIO_EM4WU5/I2C0_SCL#6/LES_ALTEX7/US0_CS#0/US0_TX#3"/>
+<wire x1="241.3" y1="91.44" x2="248.92" y2="91.44" width="0.1524" layer="91"/>
+<label x="243.84" y="91.44" size="1.778" layer="95"/>
+</segment>
 <segment>
 <pinref part="JIOH" gate="G$1" pin="3"/>
@@
 <label x="35.56" y="218.44" size="1.778" layer="95"/>
 </segment>
-<segment>
-<pinref part="MCU" gate="F" pin="PF1/DBG_SWDIO#0,1,2,3/GPIO_EM4WU3/I2C0_SCL#5/LETIM0_OUT1#2/LEU0_RX#3/TIM0_CC1#5/US1_CS#2"/>
-<wire x1="241.3" y1="111.76" x2="248.92" y2="111.76" width="0.1524" layer="91"/>
-<label x="243.84" y="111.76" size="1.778" layer="95"/>
-</segment>
-</net>
+</net>

Commit message: layout wires, needs refine
Connections:
- removed net N$3: JIOL.1
- new net LEU0_RX_2: JIOL.1, MCUE.PE15/LEU0_RX#2/TIM3_CC1
- new net LEU0_TX_2: JIOL.2, MCUE.PE14/LEU0_TX#2/TIM3_CC0
Changed lines of the file:
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@@
 </busses>
 <nets>
-<net name="N$3" class="0">
-<segment>
-<pinref part="JIOL" gate="G$1" pin="1"/>
-<wire x1="33.02" y1="182.88" x2="40.64" y2="182.88" width="0.1524" layer="91"/>
-</segment>
-</net>
 <net name="3.3V" class="0">
 <segment>
@@
 </segment>
 </net>
+<net name="LEU0_RX_2" class="0">
+<segment>
+<pinref part="MCU" gate="E" pin="PE15/LEU0_RX#2/TIM3_CC1"/>
+<wire x1="241.3" y1="96.52" x2="248.92" y2="96.52" width="0.1524" layer="91"/>
+<label x="243.84" y="96.52" size="1.778" layer="95"/>
+</segment>
+<segment>
+<pinref part="JIOL" gate="G$1" pin="1"/>
+<wire x1="33.02" y1="182.88" x2="40.64" y2="182.88" width="0.1524" layer="91"/>
+<label x="35.56" y="182.88" size="1.778" layer="95"/>
+</segment>
+</net>
+<net name="LEU0_TX_2" class="0">
+<segment>
+<pinref part="MCU" gate="E" pin="PE14/LEU0_TX#2/TIM3_CC0"/>
+<wire x1="241.3" y1="93.98" x2="248.92" y2="93.98" width="0.1524" layer="91"/>
+<label x="243.84" y="93.98" size="1.778" layer="95"/>
+</segment>
+<segment>
+<pinref part="JIOL" gate="G$1" pin="2"/>
+<wire x1="33.02" y1="185.42" x2="40.64" y2="185.42" width="0.1524" layer="91"/>
+<label x="35.56" y="185.42" size="1.778" layer="95"/>
+</segment>
+</net>
