File: efm32core.brd (EAGLE design)
At the start: 52.1 x 53.3 mm, 66 parts, among them Q1 MMBT5088, U3 USD-SOCKETNEW, X1 48.0MHz, Y1 32.768kHz

Commit message: optimize
Routing:
- net 3.3V: track 187.6 -> 193.0 mm
- net I2C0_SDA: track 41.5 -> 44.5 mm, vias 0 -> 2
- net I2C0_SCL: track 40.7 -> 41.8 mm
- net PA2: track 52.2 -> 51.8 mm, vias 0 -> 2
Changed lines of the file:
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@@
 <wire x1="33.77" y1="27.086" x2="33.782" y2="27.098" width="0.2032" layer="1"/>
 <wire x1="33.782" y1="27.098" x2="33.782" y2="29.376" width="0.2032" layer="1"/>
-<wire x1="25.484" y1="45.466" x2="27.178" y2="45.466" width="0.3048" layer="1"/>
-<wire x1="27.178" y1="45.466" x2="28.067" y2="44.577" width="0.3048" layer="1"/>
-<via x="28.067" y="44.577" extent="1-16" drill="0.7" shape="square"/>
-<wire x1="28.067" y1="44.577" x2="28.067" y2="39.37" width="0.3048" layer="16"/>
-<wire x1="28.067" y1="39.37" x2="28.067" y2="32.385" width="0.3048" layer="16"/>
-<wire x1="28.067" y1="32.385" x2="26.67" y2="30.988" width="0.3048" layer="16"/>
-<wire x1="26.67" y1="30.988" x2="23.876" y2="30.988" width="0.3048" layer="16"/>
-<wire x1="23.876" y1="30.988" x2="23.114" y2="30.226" width="0.3048" layer="16"/>
-<wire x1="23.114" y1="30.226" x2="23.114" y2="28.956" width="0.3048" layer="16"/>
+<wire x1="25.484" y1="45.466" x2="28.067" y2="45.466" width="0.3048" layer="1"/>
+<via x="28.067" y="45.466" extent="1-16" drill="0.7" shape="square"/>
 <wire x1="33.02" y1="21.336" x2="33.02" y2="21.59" width="0.4064" layer="1"/>
 <wire x1="25.781" y1="28.956" x2="33.02" y2="21.717" width="0.3048" layer="1"/>
@@
 <wire x1="34.167" y1="39.366" x2="34.163" y2="39.37" width="0.3048" layer="1"/>
 <via x="34.163" y="39.37" extent="1-16" drill="0.7" shape="square"/>
-<wire x1="34.163" y1="39.37" x2="28.067" y2="39.37" width="0.3048" layer="16"/>
 <wire x1="39.128" y1="37.116" x2="39.128" y2="34.556" width="0.3048" layer="1"/>
 <wire x1="39.128" y1="34.556" x2="38.354" y2="33.782" width="0.3048" layer="1"/>
@@
 <wire x1="14.224" y1="18.288" x2="17.272" y2="21.336" width="0.3048" layer="16"/>
 <wire x1="17.272" y1="21.336" x2="33.02" y2="21.336" width="0.3048" layer="16"/>
+<wire x1="23.114" y1="28.956" x2="23.114" y2="43.561" width="0.3048" layer="16"/>
+<wire x1="23.114" y1="43.561" x2="25.019" y2="45.466" width="0.3048" layer="16"/>
+<wire x1="34.163" y1="39.37" x2="30.48" y2="39.37" width="0.3048" layer="16"/>
+<wire x1="30.48" y1="39.37" x2="28.067" y2="41.783" width="0.3048" layer="16"/>
+<wire x1="28.067" y1="41.783" x2="28.067" y2="45.466" width="0.3048" layer="16"/>
+<wire x1="25.019" y1="45.466" x2="28.067" y2="45.466" width="0.3048" layer="16"/>
 <wire x1="37.878" y1="39.366" x2="40.982" y2="42.926" width="0" layer="19" extent="1-1"/>
 </signal>
@@
 <wire x1="37.846" y1="15.494" x2="39.751" y2="13.589" width="0.2032" layer="1"/>
 <wire x1="39.751" y1="13.589" x2="41.021" y2="13.589" width="0.2032" layer="1"/>
-<wire x1="41.021" y1="13.589" x2="42.545" y2="12.065" width="0.2032" layer="1"/>
-<wire x1="42.545" y1="12.065" x2="42.545" y2="11.303" width="0.2032" layer="1"/>
-<wire x1="42.545" y1="11.303" x2="43.053" y2="10.795" width="0.2032" layer="1"/>
+<wire x1="41.021" y1="13.589" x2="43.053" y2="11.557" width="0.2032" layer="1"/>
+<wire x1="43.053" y1="11.557" x2="43.053" y2="10.795" width="0.2032" layer="1"/>
 <via x="43.053" y="10.795" extent="1-16" drill="0.381"/>
 <wire x1="43.053" y1="10.795" x2="43.053" y2="9.906" width="0.2032" layer="16"/>
@@
 <contactref element="R7" pad="1"/>
 <wire x1="27.27" y1="25.086" x2="26.476" y2="25.086" width="0.2032" layer="1"/>
-<wire x1="30.607" y1="33.655" x2="31.115" y2="34.163" width="0.2032" layer="1"/>
-<wire x1="31.115" y1="34.163" x2="31.115" y2="38.1" width="0.2032" layer="1"/>
-<wire x1="31.115" y1="38.1" x2="34.544" y2="41.529" width="0.2032" layer="1"/>
-<wire x1="34.544" y1="41.529" x2="38.227" y2="41.529" width="0.2032" layer="1"/>
 <wire x1="38.227" y1="41.529" x2="38.628" y2="41.128" width="0.2032" layer="1"/>
 <wire x1="38.628" y1="41.128" x2="38.628" y2="41.116" width="0.2032" layer="1"/>
@@
 <wire x1="38.608" y1="44.45" x2="39.028" y2="44.45" width="0.2032" layer="1"/>
 <wire x1="39.028" y1="44.45" x2="39.282" y2="44.704" width="0.2032" layer="1"/>
-<wire x1="30.607" y1="33.655" x2="22.606" y2="33.655" width="0.2032" layer="1"/>
-<wire x1="22.606" y1="33.655" x2="19.558" y2="30.607" width="0.2032" layer="1"/>
-<wire x1="19.558" y1="30.607" x2="19.558" y2="28.956" width="0.2032" layer="1"/>
 <wire x1="19.558" y1="28.956" x2="21.844" y2="26.67" width="0.2032" layer="1"/>
 <wire x1="21.844" y1="26.67" x2="24.892" y2="26.67" width="0.2032" layer="1"/>
 <wire x1="26.476" y1="25.086" x2="24.892" y2="26.67" width="0.2032" layer="1"/>
+<wire x1="19.558" y1="28.956" x2="19.558" y2="32.385" width="0.2032" layer="1"/>
+<wire x1="19.558" y1="32.385" x2="22.479" y2="35.306" width="0.2032" layer="1"/>
+<wire x1="22.479" y1="35.306" x2="24.638" y2="35.306" width="0.2032" layer="1"/>
+<wire x1="24.638" y1="35.306" x2="27.305" y2="37.973" width="0.2032" layer="1"/>
+<wire x1="27.305" y1="37.973" x2="27.305" y2="41.402" width="0.2032" layer="1"/>
+<wire x1="27.305" y1="41.402" x2="29.464" y2="43.561" width="0.2032" layer="1"/>
+<via x="29.464" y="43.561" extent="1-16" drill="0.381"/>
+<wire x1="29.464" y1="43.561" x2="36.195" y2="43.561" width="0.2032" layer="16"/>
+<via x="36.195" y="43.561" extent="1-16" drill="0.381"/>
+<wire x1="36.195" y1="43.561" x2="37.084" y2="42.66" width="0.2032" layer="1"/>
+<wire x1="37.084" y1="42.66" x2="38.628" y2="41.116" width="0.2032" layer="1"/>
 </signal>
 <signal name="LEU1_RX">
@@
 <via x="39.116" y="40.005" extent="1-16" drill="0.381"/>
 <wire x1="39.116" y1="40.005" x2="39.116" y2="36.83" width="0.2032" layer="16"/>
-<wire x1="39.116" y1="36.83" x2="36.83" y2="34.544" width="0.2032" layer="16"/>
+<wire x1="39.116" y1="36.83" x2="38.481" y2="36.195" width="0.2032" layer="16"/>
 <wire x1="27.27" y1="24.586" x2="26.214" y2="24.586" width="0.2032" layer="1"/>
-<via x="30.226" y="34.544" extent="1-16" drill="0.381"/>
-<wire x1="30.226" y1="34.544" x2="36.83" y2="34.544" width="0.2032" layer="16"/>
-<wire x1="30.226" y1="34.544" x2="22.86" y2="34.544" width="0.2032" layer="1"/>
-<wire x1="22.86" y1="34.544" x2="19.05" y2="30.734" width="0.2032" layer="1"/>
-<wire x1="19.05" y1="30.734" x2="19.05" y2="28.702" width="0.2032" layer="1"/>
+<via x="24.13" y="36.195" extent="1-16" drill="0.381"/>
+<wire x1="24.13" y1="36.195" x2="38.481" y2="36.195" width="0.2032" layer="16"/>
+<wire x1="24.13" y1="36.195" x2="22.733" y2="36.195" width="0.2032" layer="1"/>
+<wire x1="22.733" y1="36.195" x2="19.05" y2="32.512" width="0.2032" layer="1"/>
+<wire x1="19.05" y1="32.512" x2="19.05" y2="28.702" width="0.2032" layer="1"/>
 <wire x1="19.05" y1="28.702" x2="21.59" y2="26.162" width="0.2032" layer="1"/>
 <wire x1="21.59" y1="26.162" x2="24.638" y2="26.162" width="0.2032" layer="1"/>
@@
 <wire x1="28.448" y1="25.4" x2="28.194" y2="25.654" width="0.2032" layer="1"/>
 <wire x1="28.194" y1="25.654" x2="26.67" y2="25.654" width="0.2032" layer="1"/>
-<wire x1="22.86" y1="33.147" x2="43.053" y2="33.147" width="0.2032" layer="1"/>
-<wire x1="43.053" y1="33.147" x2="47.027" y2="37.121" width="0.2032" layer="1"/>
-<wire x1="47.027" y1="37.121" x2="47.027" y2="43.412" width="0.2032" layer="1"/>
-<wire x1="22.86" y1="33.147" x2="20.066" y2="30.353" width="0.2032" layer="1"/>
-<wire x1="20.066" y1="30.353" x2="20.066" y2="29.21" width="0.2032" layer="1"/>
 <wire x1="20.066" y1="29.21" x2="22.098" y2="27.178" width="0.2032" layer="1"/>
 <wire x1="22.098" y1="27.178" x2="25.146" y2="27.178" width="0.2032" layer="1"/>
 <wire x1="25.146" y1="27.178" x2="26.67" y2="25.654" width="0.2032" layer="1"/>
+<wire x1="20.066" y1="29.21" x2="20.066" y2="32.258" width="0.2032" layer="1"/>
+<wire x1="20.066" y1="32.258" x2="22.606" y2="34.798" width="0.2032" layer="1"/>
+<wire x1="22.606" y1="34.798" x2="24.892" y2="34.798" width="0.2032" layer="1"/>
+<wire x1="24.892" y1="34.798" x2="27.813" y2="37.719" width="0.2032" layer="1"/>
+<wire x1="27.813" y1="37.719" x2="27.813" y2="40.132" width="0.2032" layer="1"/>
+<wire x1="27.813" y1="40.132" x2="29.591" y2="41.91" width="0.2032" layer="1"/>
+<via x="29.591" y="41.91" extent="1-16" drill="0.381"/>
+<wire x1="29.591" y1="41.91" x2="46.736" y2="41.91" width="0.2032" layer="16"/>
+<via x="46.736" y="41.91" extent="1-16" drill="0.381"/>
+<wire x1="46.736" y1="41.91" x2="47.027" y2="42.201" width="0.2032" layer="1"/>
+<wire x1="47.027" y1="42.201" x2="47.027" y2="43.412" width="0.2032" layer="1"/>
 </signal>
 <signal name="3.3V-BLE">
