File: efm32core.brd (EAGLE design)
At the start: 52.1 x 53.3 mm, 66 parts, among them Q1 MMBT5088, U3 USD-SOCKETNEW, X1 48.0MHz, Y1 32.768kHz

Commit message: almost done
Parts:
- removed R11: 470, SparkFun-Resistors:0603-RES
- moved C8 0.63 mm to (43.2, 18.0)
- moved S2 0.38 mm to (47.8, 45.6)
Connections:
- removed net LEU0_RX_2: JIOL.1, MCU.64
- removed net LEU0_TX_2: JIOL.2, MCU.63
- removed net N$10: MCU.54
- removed net N$17: JEX.11
- removed net N$18: JEX.13
- removed net N$19: Q1.1, R11.2
- removed net N$20: JEX.15
- removed net SWCLK: JEX.12, MCU.49
- removed net SWIO: JEX.14, MCU.50
- removed net SWO: JEX.16, MCU.51
- new net IO2: JEX.12, JIOL.3, MCU.44
- new net IO3: JEX.10, JEX.9, JIOL.4, MCU.43
- new net IO4: JIOL.5, MCU.51
- new net IO5: JIOL.6, MCU.54
- new net IO6: JIOL.7, MCU.63
- new net IO7: JIOL.8, MCU.64
- new net PD6: JEX.1, MCU.34
- new net PD7: JEX.2, MCU.35
- new net SWCLK/LEU0_TX_3: JEX.14, JIOL.2, MCU.49
- new net SWIO/LEU0_RX_3: JEX.16, JIOL.1, MCU.50
- net GND: now also JEX.3
- net IO10: now also Q1.1; no longer R11.1
- net LEU1_RX: now also JEX.8
- net LEU1_TX: now also JEX.6
- net PD8: now also JEX.4
Routing:
- net LEU0_RX_2: track 58.9 -> 0.00 mm, vias 2 -> 0
- net IO3: track 0.00 -> 46.7 mm, vias 0 -> 1
- net IO2: track 0.00 -> 38.9 mm, vias 0 -> 1
- net SWCLK/LEU0_TX_3: track 0.00 -> 37.9 mm, vias 0 -> 1
- net LEU0_TX_2: track 37.4 -> 0.00 mm, vias 2 -> 0
- net SWIO/LEU0_RX_3: track 0.00 -> 37.2 mm
- net IO7: track 0.00 -> 32.5 mm, vias 0 -> 2
- net IO6: track 0.00 -> 31.4 mm, vias 0 -> 2
- net IO4: track 0.00 -> 27.3 mm
- net IO5: track 0.00 -> 26.4 mm
- net PD6: track 0.00 -> 19.1 mm, vias 0 -> 1
- net SWCLK: track 15.3 -> 0.00 mm
- net LEU1_RX: track 0.00 -> 14.3 mm, vias 0 -> 1
- net SWO: track 14.0 -> 0.00 mm
- net PD7: track 0.00 -> 13.1 mm, vias 0 -> 1
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
Commit message: refine
Parts:
- added JSER: (no value), SparkFun-Connectors:1X04-1.27MM
Connections:
- net GND: now also JEX.5, JEX.7
- net US2_CLK: now also JSER.2
- net US2_CS: now also JSER.4
- net US2_RX: now also JSER.1
- net US2_TX: now also JSER.3
Routing:
- net BLE-USB+: track 32.9 -> 44.2 mm, vias 1 -> 2
- net US2_CS: track 21.8 -> 27.2 mm
- net US2_RX: track 25.8 -> 31.1 mm
- net US2_TX: track 22.0 -> 27.3 mm
- net US2_CLK: track 24.4 -> 29.3 mm
- net GND: track 36.0 -> 32.4 mm, vias 73 -> 85
- net PA2: track 51.5 -> 50.9 mm
- net VDD: track 42.4 -> 41.9 mm
Other:
- outline, holes or cut-outs redrawn

Commit message: refine
Routing:
- net US0_CS: track 45.0 -> 43.4 mm
- net 3.3V: track 213.2 -> 212.4 mm
- net US0_CLK: track 49.7 -> 49.0 mm
Other:
- outline, holes or cut-outs redrawn
